File: kicad/dds_analog.sch (KiCad schematic (older format))
At the start: 50 parts, among them J1 Conn_Coaxial, U1 AD9954, U2 OPA859xDSG, X1 ASE-xxxMHz

Commit message: removed frontent/amp test circuit
This circuit had shared the PCB for cost reasons.
Parts:
- U1: symbol obbo_IC:AD9954 -> siggen-v1-rescue:AD9954-obbo_IC
Changed lines of the file:
@@
 $Descr A4 11693 8268
 encoding utf-8
-Sheet 2 5
+Sheet 2 4
 Title ""
 Date ""
@@
 $EndComp
 $Comp
-L obbo_IC:AD9954 U?
+L siggen-v1-rescue:AD9954-obbo_IC U?
 U 1 1 6246FE03
 P 4050 3650

Commit message: renamed objects that had '-v1' in their names
Parts:
- U1: symbol siggen-v1-rescue:AD9954-obbo_IC -> siggen-rescue:AD9954-obbo_IC
Changed lines of the file:
@@
 $EndComp
 $Comp
-L siggen-v1-rescue:AD9954-obbo_IC U?
+L siggen-rescue:AD9954-obbo_IC U?
 U 1 1 6246FE03
 P 4050 3650
